Commit message: Modified the control node -  debugged the motion planner

File: models/panda_description/levi_panda.urdf (robot description, URDF)
Before this commit: robot panda, 9 links, 8 joints
Links:
- added link levitator, mass 1.724; collision mesh filename=/models/levitator/levitator.STL scale=0.001 0.001 0.001; visual mesh filename=/models/levitator/levitator.STL scale=0.001 0.001 0.001
Joints:
- added joint levitator_joint: type fixed, parent panda_link8, child levitator, origin xyz=0.0376181 -0.0376181 0.1358 rpy=-1.5707963267948966 0 -2.356194490192344
